File: board/LoRaKid/LoRaKid.kicad_sch (KiCad schematic)
At the start: 10 parts, among them SW1_ON_OFF1 SW_Push, SW2_LEFT1 SW_Push, SW3_RIGHT1 SW_Push, SW4 SW_Push, SW5 SW_Push, SW6 SW_Push, SW7 SW_Push, SW8 SW_Push, SW9 SW_Push

Commit message: update board design
Parts:
- added BZ1: Buzzer, Buzzer_Beeper:Buzzer_12x9.5RM7.6, symbol Device:Buzzer
- added Q1: NPN, Package_TO_SOT_THT:TO-92_Inline, symbol Transistor_BJT:2N3904
- added R1: 470, Resistor_SMD:R_0805_2012Metric_Pad1.20x1.40mm_HandSolder, symbol Device:R
- added R2: 4,7 k, Resistor_SMD:R_0805_2012Metric_Pad1.20x1.40mm_HandSolder, symbol Device:R
- added USB1: Conn_01x04_Pin, Connector_PinSocket_2.54mm:PinSocket_1x04_P2.54mm_Vertical, symbol Connector:Conn_01x04_Pin
- SW1_ON_OFF1, SW2_LEFT1, SW3_RIGHT1, SW4, SW5, SW6, SW7, SW8, SW9: footprint (none) -> Button_Switch_SMD:SW_SPST_Omron_B3FS-100xP
Connections:
- net GND: now also Q1.1 (E), R2.2, USB1.4 (Pin_4)
- net +3.3V: now reaches U1.2 (3V3)
- net +3.3V: now also U1.3 (3V3), BZ1.1 (+)
- net at U1.20 (5V): now also USB1.1 (Pin_1)
- net at U1.30 (GPIO33): now also R1.1
- new net: Q1.2 (B), R1.2, R2.1
- new net: BZ1.2 (-), Q1.3 (C)

Commit message: update board layout
Parts:
- added BAT1: Conn_01x02_Pin, Connector_JST:JST_PH_B2B-PH-K_1x02_P2.00mm_Vertical, symbol Connector:Conn_01x02_Pin
- added J1: Conn_01x02_Pin, Connector_PinHeader_2.54mm:PinHeader_1x02_P2.54mm_Vertical, symbol Connector:Conn_01x02_Pin
Connections:
- net GND: now also BAT1.1 (Pin_1), J1.1 (Pin_1)
- new net: BAT1.2 (Pin_2), J1.2 (Pin_2)
